File: base/PCB/universal16.sch (KiCad schematic (older format))
At the start: 105 parts, among them J1 Conn_01x04, J10 Conn_01x01, J11 Conn_01x01, J12 Conn_01x01, J13 Conn_01x01, J14 Conn_01x03, J2 Conn_01x04, J3 Conn_01x03, J4 Conn_01x03, J5 Conn_01x04, J6 Conn_01x04, J7 Conn_01x03, J8 Conn_01x03, J9 Conn_01x03, SW1 SW_Push, SW10 SW_Push, SW11 SW_Push, SW12 SW_Push, SW13 SW_Push, SW14 SW_Push, SW15 SW_Push, SW16 SW_Push, SW2 SW_Push, SW3 SW_Push, SW4 SW_Push, SW5 SW_Push, SW6 SW_Push, SW7 SW_Push, SW8 SW_Push, SW9 SW_Push, U1 ProMicro

Commit message: update some footprints
Parts:
- J1, J2, J5, J6: footprint Connector_PinSocket_2.54mm:PinSocket_1x04_P2.54mm_Vertical -> myfootplint:PinSocket_1x04_P2.54mm_Vertical
- J14, J3, J4, J7, J8, J9: footprint Connector_PinSocket_2.54mm:PinSocket_1x03_P2.54mm_Vertical -> myfootplint:PinSocket_1x03_P2.54mm_Vertical
Changed lines of the file:
@@
 F 0 "J7" H 1730 5192 50  0000 L CNN
 F 1 "Conn_01x03" H 1730 5101 50  0000 L CNN
-F 2 "Connector_PinSocket_2.54mm:PinSocket_1x03_P2.54mm_Vertical" H 1650 5150 50  0001 C CNN
+F 2 "myfootplint:PinSocket_1x03_P2.54mm_Vertical" H 1650 5150 50  0001 C CNN
 F 3 "~" H 1650 5150 50  0001 C CNN
 	1    1650 5150
@@
 F 0 "J9" H 1730 5692 50  0000 L CNN
 F 1 "Conn_01x03" H 1730 5601 50  0000 L CNN
-F 2 "Connector_PinSocket_2.54mm:PinSocket_1x03_P2.54mm_Vertical" H 1650 5650 50  0001 C CNN
+F 2 "myfootplint:PinSocket_1x03_P2.54mm_Vertical" H 1650 5650 50  0001 C CNN
 F 3 "~" H 1650 5650 50  0001 C CNN
 	1    1650 5650
@@
 F 0 "J1" H 1280 2042 50  0000 L CNN
 F 1 "Conn_01x04" H 1280 1951 50  0000 L CNN
-F 2 "Connector_PinSocket_2.54mm:PinSocket_1x04_P2.54mm_Vertical" H 1200 2050 50  0001 C CNN
+F 2 "myfootplint:PinSocket_1x04_P2.54mm_Vertical" H 1200 2050 50  0001 C CNN
 F 3 "~" H 1200 2050 50  0001 C CNN
 	1    1200 2050
@@
 F 0 "J2" H 2880 2042 50  0000 L CNN
 F 1 "Conn_01x04" H 2880 1951 50  0000 L CNN
-F 2 "Connector_PinSocket_2.54mm:PinSocket_1x04_P2.54mm_Vertical" H 2800 2050 50  0001 C CNN
+F 2 "myfootplint:PinSocket_1x04_P2.54mm_Vertical" H 2800 2050 50  0001 C CNN
 F 3 "~" H 2800 2050 50  0001 C CNN
 	1    2800 2050
@@
 F 0 "J6" H 2880 3292 50  0000 L CNN
 F 1 "Conn_01x04" H 2880 3201 50  0000 L CNN
-F 2 "Connector_PinSocket_2.54mm:PinSocket_1x04_P2.54mm_Vertical" H 2800 3300 50  0001 C CNN
+F 2 "myfootplint:PinSocket_1x04_P2.54mm_Vertical" H 2800 3300 50  0001 C CNN
 F 3 "~" H 2800 3300 50  0001 C CNN
 	1    2800 3300
@@
 F 0 "J5" H 1280 3292 50  0000 L CNN
 F 1 "Conn_01x04" H 1280 3201 50  0000 L CNN
-F 2 "Connector_PinSocket_2.54mm:PinSocket_1x04_P2.54mm_Vertical" H 1200 3300 50  0001 C CNN
+F 2 "myfootplint:PinSocket_1x04_P2.54mm_Vertical" H 1200 3300 50  0001 C CNN
 F 3 "~" H 1200 3300 50  0001 C CNN
 	1    1200 3300
@@
 F 0 "J8" H 1780 6592 50  0000 L CNN
 F 1 "Conn_01x03" H 1780 6501 50  0000 L CNN
-F 2 "Connector_PinSocket_2.54mm:PinSocket_1x03_P2.54mm_Vertical" H 1700 6550 50  0001 C CNN
+F 2 "myfootplint:PinSocket_1x03_P2.54mm_Vertical" H 1700 6550 50  0001 C CNN
 F 3 "~" H 1700 6550 50  0001 C CNN
 	1    1700 6550
@@
 F 0 "J3" H 4030 5192 50  0000 L CNN
 F 1 "Conn_01x03" H 4030 5101 50  0000 L CNN
-F 2 "Connector_PinSocket_2.54mm:PinSocket_1x03_P2.54mm_Vertical" H 3950 5150 50  0001 C CNN
+F 2 "myfootplint:PinSocket_1x03_P2.54mm_Vertical" H 3950 5150 50  0001 C CNN
 F 3 "~" H 3950 5150 50  0001 C CNN
 	1    3950 5150
@@
 F 0 "J4" H 4030 5692 50  0000 L CNN
 F 1 "Conn_01x03" H 4030 5601 50  0000 L CNN
-F 2 "Connector_PinSocket_2.54mm:PinSocket_1x03_P2.54mm_Vertical" H 3950 5650 50  0001 C CNN
+F 2 "myfootplint:PinSocket_1x03_P2.54mm_Vertical" H 3950 5650 50  0001 C CNN
 F 3 "~" H 3950 5650 50  0001 C CNN
 	1    3950 5650
@@
 F 0 "J14" H 4030 2792 50  0000 L CNN
 F 1 "Conn_01x03" H 4030 2701 50  0000 L CNN
-F 2 "Connector_PinSocket_2.54mm:PinSocket_1x03_P2.54mm_Vertical" H 3950 2750 50  0001 C CNN
+F 2 "myfootplint:PinSocket_1x03_P2.54mm_Vertical" H 3950 2750 50  0001 C CNN
 F 3 "~" H 3950 2750 50  0001 C CNN
 	1    3950 2750
